File: line following robot sensor circuit/photo.brd (EAGLE design)
At the start: 63.5 x 25.4 mm, 17 parts

Commit message: version 2.1
1. Added a new LCD GUI to tune the Kp, Kd, easier to setup
2. Added EEPROM library, can save the Kp, Kd data, not need to tune
again when restarting(DON’T SAVE TOO MUCH, EEPROM only 100,000 cycle
life)
3. Change the edge sensor pin to digital pin, A4, A5 is used to IIC
communication.

You also need a IIC LCD display
Parts:
- removed R1, R3, R5, R7, R9: 4.7k, adafruit:0207/7
- R2: device adafruit:0207/2V -> adafruit:0204/7
- moved R2 3.59 mm to (3.81, 20.3)
Connections:
- net N$10: no longer R5.1
- net N$15: no longer R7.1
- net N$19: no longer R9.1
- net N$2: no longer R1.2, R3.2, R5.2, R7.2, R9.2
- net N$3: no longer R3.1
- net N$8: no longer R1.1
Routing:
- net N$2: track 78.7 -> 63.5 mm
- net N$10: track 50.8 -> 38.1 mm
- net N$15: track 66.0 -> 53.3 mm
- net N$3: track 30.5 -> 22.9 mm
- net N$8: track 12.7 -> 7.62 mm
- net N$4: track 2.54 -> 5.08 mm
Changed lines of the file:
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@@
 <attribute name="VALUE" x="4.445" y="11.176" size="1.27" layer="27" ratio="10" rot="R270"/>
 </element>
-<element name="R1" library="adafruit" package="0207/7" value="4.7k" x="10.16" y="13.97" smashed="yes" rot="R90">
-<attribute name="VALUE" x="10.7188" y="11.684" size="1.27" layer="27" ratio="10" rot="R90"/>
-</element>
-<element name="R2" library="adafruit" package="0207/2V" value="100" x="1.27" y="17.78" smashed="yes">
-<attribute name="VALUE" x="1.524" y="18.4912" size="1.27" layer="27" ratio="10"/>
+<element name="R2" library="adafruit" package="0204/7" value="100" x="3.81" y="20.32" smashed="yes">
+<attribute name="VALUE" x="4.064" y="21.0312" size="1.27" layer="27" ratio="10"/>
 </element>
 <element name="LED2" library="adafruit" package="LED3MM" value="" x="19.05" y="17.78" smashed="yes">
@@
 <attribute name="VALUE" x="17.145" y="11.176" size="1.27" layer="27" ratio="10" rot="R270"/>
 </element>
-<element name="R3" library="adafruit" package="0207/7" value="4.7k" x="22.86" y="13.97" smashed="yes" rot="R90">
-<attribute name="VALUE" x="23.4188" y="11.684" size="1.27" layer="27" ratio="10" rot="R90"/>
-</element>
 <element name="LED3" library="adafruit" package="LED3MM" value="" x="31.75" y="17.78" smashed="yes">
 <attribute name="VALUE" x="33.655" y="16.129" size="1.27" layer="27" ratio="10"/>
@@
 <attribute name="OC_FARNELL" value="unknown" x="34.29" y="12.7" size="1.778" layer="27" rot="R270" display="off"/>
 <attribute name="VALUE" x="29.845" y="11.176" size="1.27" layer="27" ratio="10" rot="R270"/>
-</element>
-<element name="R5" library="adafruit" package="0207/7" value="4.7k" x="35.56" y="13.97" smashed="yes" rot="R90">
-<attribute name="VALUE" x="36.1188" y="11.684" size="1.27" layer="27" ratio="10" rot="R90"/>
 </element>
 <element name="LED4" library="adafruit" package="LED3MM" value="" x="44.45" y="17.78" smashed="yes">
@@
 <attribute name="VALUE" x="42.545" y="11.176" size="1.27" layer="27" ratio="10" rot="R270"/>
 </element>
-<element name="R7" library="adafruit" package="0207/7" value="4.7k" x="48.26" y="13.97" smashed="yes" rot="R90">
-<attribute name="VALUE" x="48.8188" y="11.684" size="1.27" layer="27" ratio="10" rot="R90"/>
-</element>
 <element name="LED5" library="adafruit" package="LED3MM" value="" x="57.15" y="17.78" smashed="yes">
 <attribute name="VALUE" x="59.055" y="16.129" size="1.27" layer="27" ratio="10"/>
@@
 <attribute name="OC_FARNELL" value="unknown" x="59.69" y="12.7" size="1.778" layer="27" rot="R270" display="off"/>
 <attribute name="VALUE" x="55.245" y="11.176" size="1.27" layer="27" ratio="10" rot="R270"/>
-</element>
-<element name="R9" library="adafruit" package="0207/7" value="4.7k" x="53.34" y="13.97" smashed="yes" rot="R90">
-<attribute name="VALUE" x="53.8988" y="11.684" size="1.27" layer="27" ratio="10" rot="R90"/>
 </element>
 <element name="SV1" library="con-lstb" package="MA07-1" value="" x="0" y="7.62" smashed="yes" rot="R270">
@@
 <signals>
 <signal name="N$8">
-<contactref element="R1" pad="1"/>
 <contactref element="T1" pad="C"/>
 <contactref element="SV1" pad="3"/>
 <wire x1="0" y1="10.16" x2="5.08" y2="10.16" width="1.016" layer="16"/>
-<wire x1="5.08" y1="10.16" x2="10.16" y2="10.16" width="1.016" layer="16"/>
 <wire x1="5.08" y1="12.7" x2="5.08" y2="10.16" width="1.016" layer="16"/>
 </signal>
 <signal name="N$3">
-<contactref element="R3" pad="1"/>
 <contactref element="T2" pad="C"/>
 <contactref element="SV1" pad="4"/>
 <wire x1="0" y1="7.62" x2="17.78" y2="7.62" width="1.016" layer="16"/>
-<wire x1="17.78" y1="7.62" x2="22.86" y2="7.62" width="1.016" layer="16"/>
-<wire x1="22.86" y1="7.62" x2="22.86" y2="10.16" width="1.016" layer="16"/>
-<wire x1="17.78" y1="12.7" x2="17.78" y2="7.62" width="1.016" layer="16"/>
+<wire x1="17.78" y1="7.62" x2="17.78" y2="12.7" width="1.016" layer="16"/>
 </signal>
 <signal name="N$10">
-<contactref element="R5" pad="1"/>
 <contactref element="T3" pad="C"/>
 <contactref element="SV1" pad="5"/>
-<wire x1="0" y1="5.08" x2="35.56" y2="5.08" width="1.016" layer="16"/>
-<wire x1="35.56" y1="5.08" x2="35.56" y2="7.62" width="1.016" layer="16"/>
-<wire x1="35.56" y1="7.62" x2="35.56" y2="10.16" width="1.016" layer="16"/>
-<wire x1="30.48" y1="12.7" x2="30.48" y2="7.62" width="1.016" layer="16"/>
-<wire x1="30.48" y1="7.62" x2="35.56" y2="7.62" width="1.016" layer="16"/>
+<wire x1="30.48" y1="12.7" x2="30.48" y2="5.08" width="1.016" layer="16"/>
+<wire x1="30.48" y1="5.08" x2="0" y2="5.08" width="1.016" layer="16"/>
 </signal>
 <signal name="N$15">
-<contactref element="R7" pad="1"/>
 <contactref element="T4" pad="C"/>
 <contactref element="SV1" pad="6"/>
-<wire x1="48.26" y1="10.16" x2="48.26" y2="7.62" width="1.016" layer="16"/>
-<wire x1="48.26" y1="7.62" x2="48.26" y2="2.54" width="1.016" layer="16"/>
-<wire x1="48.26" y1="2.54" x2="0" y2="2.54" width="1.016" layer="16"/>
-<wire x1="43.18" y1="12.7" x2="43.18" y2="7.62" width="1.016" layer="16"/>
-<wire x1="43.18" y1="7.62" x2="48.26" y2="7.62" width="1.016" layer="16"/>
+<wire x1="0" y1="2.54" x2="43.18" y2="2.54" width="1.016" layer="16"/>
+<wire x1="43.18" y1="2.54" x2="43.18" y2="12.7" width="1.016" layer="16"/>
 </signal>
 <signal name="N$17">
@@
 </signal>
 <signal name="N$19">
-<contactref element="R9" pad="1"/>
 <contactref element="T5" pad="C"/>
 <contactref element="SV1" pad="7"/>
-<wire x1="53.34" y1="10.16" x2="53.34" y2="0" width="1.016" layer="16"/>
-<wire x1="53.34" y1="0" x2="0" y2="0" width="1.016" layer="16"/>
-<wire x1="55.88" y1="12.7" x2="55.88" y2="10.16" width="1.016" layer="16"/>
-<wire x1="55.88" y1="10.16" x2="53.34" y2="10.16" width="1.016" layer="16"/>
+<wire x1="0" y1="0" x2="55.88" y2="0" width="1.016" layer="16"/>
+<wire x1="55.88" y1="0" x2="55.88" y2="12.7" width="1.016" layer="16"/>
 </signal>
 <signal name="N$2">
 <contactref element="LED5" pad="A"/>
-<wire x1="55.88" y1="20.32" x2="53.34" y2="20.32" width="1.016" layer="16"/>
-<wire x1="53.34" y1="20.32" x2="48.26" y2="20.32" width="1.016" layer="16"/>
-<wire x1="48.26" y1="20.32" x2="43.18" y2="20.32" width="1.016" layer="16"/>
-<wire x1="43.18" y1="20.32" x2="35.56" y2="20.32" width="1.016" layer="16"/>
-<wire x1="35.56" y1="20.32" x2="30.48" y2="20.32" width="1.016" layer="16"/>
-<wire x1="30.48" y1="20.32" x2="22.86" y2="20.32" width="1.016" layer="16"/>
-<wire x1="22.86" y1="20.32" x2="17.78" y2="20.32" width="1.016" layer="16"/>
-<wire x1="17.78" y1="20.32" x2="10.16" y2="20.32" width="1.016" layer="16"/>
-<wire x1="10.16" y1="20.32" x2="5.08" y2="20.32" width="1.016" layer="16"/>
-<wire x1="5.08" y1="17.78" x2="2.54" y2="17.78" width="1.016" layer="16"/>
+<wire x1="55.88" y1="20.32" x2="43.18" y2="20.32" width="1.016" layer="16"/>
+<wire x1="43.18" y1="20.32" x2="30.48" y2="20.32" width="1.016" layer="16"/>
+<wire x1="30.48" y1="20.32" x2="17.78" y2="20.32" width="1.016" layer="16"/>
 <wire x1="55.88" y1="17.78" x2="55.88" y2="20.32" width="1.016" layer="16"/>
 <contactref element="LED4" pad="A"/>
 <contactref element="LED3" pad="A"/>
 <contactref element="LED2" pad="A"/>
-<contactref element="LED1" pad="A"/>
-<contactref element="R1" pad="2"/>
-<contactref element="R3" pad="2"/>
-<contactref element="R5" pad="2"/>
-<contactref element="R7" pad="2"/>
-<contactref element="R9" pad="2"/>
-<contactref element="R2" pad="2"/>
-<wire x1="5.08" y1="20.32" x2="5.08" y2="17.78" width="1.016" layer="16"/>
 <wire x1="17.78" y1="17.78" x2="17.78" y2="20.32" width="1.016" layer="16"/>
 <wire x1="30.48" y1="17.78" x2="30.48" y2="20.32" width="1.016" layer="16"/>
 <wire x1="43.18" y1="17.78" x2="43.18" y2="20.32" width="1.016" layer="16"/>
-<wire x1="53.34" y1="17.78" x2="53.34" y2="20.32" width="1.016" layer="16"/>
-<wire x1="48.26" y1="17.78" x2="48.26" y2="20.32" width="1.016" layer="16"/>
-<wire x1="35.56" y1="17.78" x2="35.56" y2="20.32" width="1.016" layer="16"/>
-<wire x1="22.86" y1="17.78" x2="22.86" y2="20.32" width="1.016" layer="16"/>
-<wire x1="10.16" y1="17.78" x2="10.16" y2="20.32" width="1.016" layer="16"/>
+<contactref element="R2" pad="2"/>
+<contactref element="LED1" pad="A"/>
+<wire x1="5.08" y1="17.78" x2="5.08" y2="20.32" width="1.016" layer="16"/>
+<wire x1="5.08" y1="20.32" x2="17.78" y2="20.32" width="1.016" layer="16"/>
 </signal>
 <signal name="N$4">
 <contactref element="SV1" pad="1"/>
 <contactref element="R2" pad="1"/>
-<wire x1="0" y1="15.24" x2="0" y2="17.78" width="1.016" layer="16"/>
+<wire x1="0" y1="15.24" x2="0" y2="20.32" width="1.016" layer="16"/>
 </signal>
 </signals>
+<errors>
+</errors>
 </board>
 </drawing>
